File: eSim/Examples/BJT_Biascircuit/BJT_Biascircuit.sch (KiCad schematic (older format))
At the start: 6 parts, among them Q1 eSim_NPN, U1 plot_i2

Commit message: permission and online-offline mode
Parts:
- Q1: symbol eSim_NPN -> eSim_NPN-RESCUE-BJT_Biascircuit
Changed lines of the file:
@@
 LIBS:74xx
 LIBS:cmos4000
+LIBS:eSim_Plot
 LIBS:BJT_Biascircuit-cache
 EELAYER 25 0
@@
 $EndComp
 $Comp
-L eSim_NPN Q1
+L eSim_NPN-RESCUE-BJT_Biascircuit Q1
 U 1 1 5D5CEC51
 P 5350 3200
@@
 $Comp
 L PWR_FLAG #FLG02
-U 1 1 5D5F9EDB
-P 5550 4100
-F 0 "#FLG02" H 5550 4175 50  0001 C CNN
-F 1 "PWR_FLAG" H 5550 4250 50  0000 C CNN
-F 2 "" H 5550 4100 50  0001 C CNN
-F 3 "" H 5550 4100 50  0001 C CNN
-	1    5550 4100
+U 1 1 5D665114
+P 5600 4150
+F 0 "#FLG02" H 5600 4225 50  0001 C CNN
+F 1 "PWR_FLAG" H 5600 4300 50  0000 C CNN
+F 2 "" H 5600 4150 50  0001 C CNN
+F 3 "" H 5600 4150 50  0001 C CNN
+	1    5600 4150
 	1    0    0    -1
 $EndComp
 Wire Wire Line
-	5550 4100 5550 4250
-Connection ~ 5550 4250
+	5600 4150 5600 4250
+Connection ~ 5600 4250
 $EndSCHEMATC
