File: eSim/Examples/BJT_CB_config/BJT_CB_config.sch (KiCad schematic (older format))
At the start: 6 parts, among them Q1 eSim_NPN

Commit message: permission and online-offline mode
Parts:
- Q1: symbol eSim_NPN -> eSim_NPN-RESCUE-BJT_CB_config
Changed lines of the file:
@@
 $EndComp
 $Comp
-L eSim_NPN Q1
+L eSim_NPN-RESCUE-BJT_CB_config Q1
 U 1 1 5D5CEEB2
 P 5450 3200
@@
 $Comp
 L PWR_FLAG #FLG02
-U 1 1 5D5FA04B
-P 5350 4050
-F 0 "#FLG02" H 5350 4125 50  0001 C CNN
-F 1 "PWR_FLAG" H 5350 4200 50  0000 C CNN
-F 2 "" H 5350 4050 50  0001 C CNN
-F 3 "" H 5350 4050 50  0001 C CNN
-	1    5350 4050
+U 1 1 5D665163
+P 5600 4150
+F 0 "#FLG02" H 5600 4225 50  0001 C CNN
+F 1 "PWR_FLAG" H 5600 4300 50  0000 C CNN
+F 2 "" H 5600 4150 50  0001 C CNN
+F 3 "" H 5600 4150 50  0001 C CNN
+	1    5600 4150
 	1    0    0    -1
 $EndComp
 Wire Wire Line
-	5350 4050 5350 4250
-Connection ~ 5350 4250
+	5600 4150 5600 4250
+Connection ~ 5600 4250
 $EndSCHEMATC
