File: eSim/Examples/BJT_CE_config/BJT_CE_config.sch (KiCad schematic (older format))
At the start: 6 parts, among them Q1 eSim_NPN

Commit message: permission and online-offline mode
Parts:
- Q1: symbol eSim_NPN-RESCUE-BJT_CE_config -> eSim_NPN
Changed lines of the file:
@@
 $EndComp
 $Comp
-L eSim_NPN-RESCUE-BJT_CE_config Q1
+L eSim_NPN Q1
 U 1 1 5D5CEE49
 P 5350 3200
@@
 $Comp
 L PWR_FLAG #FLG02
-U 1 1 5D5FA231
+U 1 1 5D66519A
 P 5600 4100
 F 0 "#FLG02" H 5600 4175 50  0001 C CNN
