File: eSim/src/SubcircuitLibrary/LM7812/LM7812.sch (KiCad schematic (older format))
At the start: 41 parts, among them Q1 eSim_NPN, Q10 eSim_NPN, Q11 eSim_NPN, Q12 eSim_NPN, Q13 eSim_NPN, Q14 eSim_PNP, Q15 eSim_NPN, Q16 eSim_NPN, Q17 eSim_NPN, Q2 eSim_NPN, Q3 eSim_NPN, Q4 eSim_NPN, Q5 eSim_PNP, Q6 eSim_NPN, Q7 eSim_NPN, Q8 eSim_NPN, Q9 eSim_PNP, U1 zener, U2 zener, U3 PORT

Commit message: permission and online-offline mode
Parts:
- Q1, Q10, Q11, Q12, Q13, Q15, Q16, Q17, Q2, Q3, Q4, Q6, Q7, Q8: symbol eSim_NPN -> eSim_NPN-RESCUE-LM7812-RESCUE-LM7812
- Q14, Q5, Q9: symbol eSim_PNP -> eSim_PNP-RESCUE-LM7812
Changed lines of the file:
@@
 EESchema Schematic File Version 2
+LIBS:LM7812-rescue
 LIBS:eSim_Analog
 LIBS:eSim_Devices
@@
 $EndComp
 $Comp
-L eSim_NPN Q1
+L eSim_NPN-RESCUE-LM7812-RESCUE-LM7812 Q1
 U 1 1 5CE41586
 P 1850 2350
@@
 Connection ~ 1250 2350
 $Comp
-L eSim_NPN Q2
+L eSim_NPN-RESCUE-LM7812-RESCUE-LM7812 Q2
 U 1 1 5CE41D6C
 P 2650 3350
@@
 $EndComp
 $Comp
-L eSim_NPN Q4
+L eSim_NPN-RESCUE-LM7812-RESCUE-LM7812 Q4
 U 1 1 5CE41E26
 P 3100 4100
@@
 $EndComp
 $Comp
-L eSim_NPN Q3
+L eSim_NPN-RESCUE-LM7812-RESCUE-LM7812 Q3
 U 1 1 5CE41EFE
 P 2850 4650
@@
 Connection ~ 2750 5200
 $Comp
-L eSim_NPN Q6
+L eSim_NPN-RESCUE-LM7812-RESCUE-LM7812 Q6
 U 1 1 5CE424FB
 P 3650 4650
@@
 Connection ~ 3200 5200
 $Comp
-L eSim_NPN Q7
+L eSim_NPN-RESCUE-LM7812-RESCUE-LM7812 Q7
 U 1 1 5CE427DA
 P 3700 2750
@@
 $EndComp
 $Comp
-L eSim_NPN Q8
+L eSim_NPN-RESCUE-LM7812-RESCUE-LM7812 Q8
 U 1 1 5CE428D0
 P 3700 3400
@@
 $EndComp
 $Comp
-L eSim_NPN Q12
+L eSim_NPN-RESCUE-LM7812-RESCUE-LM7812 Q12
 U 1 1 5CE4293A
 P 4350 3000
@@
 	3600 2450 3600 2550
 $Comp
-L eSim_PNP Q5
+L eSim_PNP-RESCUE-LM7812 Q5
 U 1 1 5CE43397
 P 3450 1700
@@
 $EndComp
 $Comp
-L eSim_PNP Q9
+L eSim_PNP-RESCUE-LM7812 Q9
 U 1 1 5CE4353C
 P 4100 1700
@@
 $EndComp
 $Comp
-L eSim_NPN Q10
+L eSim_NPN-RESCUE-LM7812-RESCUE-LM7812 Q10
 U 1 1 5CE43705
 P 4100 2200
@@
 Connection ~ 2200 5200
 $Comp
-L eSim_NPN Q11
+L eSim_NPN-RESCUE-LM7812-RESCUE-LM7812 Q11
 U 1 1 5CE4439E
 P 4300 4400
@@
 $EndComp
 $Comp
-L eSim_NPN Q13
+L eSim_NPN-RESCUE-LM7812-RESCUE-LM7812 Q13
 U 1 1 5CE44419
 P 4600 4800
@@
 Connection ~ 4700 4150
 $Comp
-L eSim_PNP Q14
+L eSim_PNP-RESCUE-LM7812 Q14
 U 1 1 5CE45652
 P 5050 3950
@@
 Connection ~ 4750 3450
 $Comp
-L eSim_NPN Q15
+L eSim_NPN-RESCUE-LM7812-RESCUE-LM7812 Q15
 U 1 1 5CE463AD
 P 5400 2150
@@
 	5850 2150 5600 2150
 $Comp
-L eSim_NPN Q16
+L eSim_NPN-RESCUE-LM7812-RESCUE-LM7812 Q16
 U 1 1 5CE4907A
 P 6550 1600
@@
 $EndComp
 $Comp
-L eSim_NPN Q17
+L eSim_NPN-RESCUE-LM7812-RESCUE-LM7812 Q17
 U 1 1 5CE4942E
 P 7300 1950
