File: eSim/src/SubcircuitLibrary/lm7805/lm7805.sch (KiCad schematic (older format))
At the start: 41 parts, among them Q1 eSim_NPN, Q10 eSim_NPN, Q11 eSim_NPN, Q12 eSim_NPN, Q13 eSim_NPN, Q14 eSim_PNP, Q15 eSim_NPN, Q16 eSim_NPN, Q17 eSim_NPN, Q2 eSim_NPN, Q3 eSim_NPN, Q4 eSim_NPN, Q5 eSim_PNP, Q6 eSim_NPN, Q7 eSim_NPN, Q8 eSim_NPN, Q9 eSim_PNP, U1 zener, U2 zener, U3 PORT

Commit message: permission and online-offline mode
Parts:
- removed Q1: eSim_NPN, symbol eSim_NPN
- added Q1: eSim_NPN, symbol eSim_NPN-RESCUE-lm7805
- Q10, Q11, Q12, Q13, Q15, Q16, Q17, Q2, Q3, Q4, Q6, Q7, Q8: symbol eSim_NPN -> eSim_NPN-RESCUE-lm7805
Connections:
- net at R1.2, U1.OUT: now also Q1.2 (B)
- net at R2.2: now also Q1.1 (C)
- net at R3.1: now also Q1.3 (E)
Changed lines of the file:
@@
 EESchema Schematic File Version 2
-LIBS:adc-dac
-LIBS:memory
-LIBS:xilinx
-LIBS:microcontrollers
-LIBS:dsp
-LIBS:microchip
-LIBS:analog_switches
-LIBS:motorola
-LIBS:texas
-LIBS:intel
-LIBS:audio
-LIBS:interface
-LIBS:digital-audio
-LIBS:philips
-LIBS:display
-LIBS:cypress
-LIBS:siliconi
-LIBS:opto
-LIBS:atmel
-LIBS:contrib
-LIBS:power
-LIBS:device
-LIBS:transistors
-LIBS:conn
-LIBS:linear
-LIBS:regul
-LIBS:74xx
-LIBS:cmos4000
+LIBS:lm7805-rescue
 LIBS:eSim_Analog
 LIBS:eSim_Devices
@@
 LIBS:eSim_Hybrid
 LIBS:eSim_Miscellaneous
+LIBS:eSim_Plot
 LIBS:eSim_Power
+LIBS:eSim_PSpice
 LIBS:eSim_Sources
 LIBS:eSim_Subckt
 LIBS:eSim_User
-LIBS:eSim_Plot
-LIBS:eSim_PSpice
 LIBS:lm7805-cache
 EELAYER 25 0
@@
 $EndComp
 $Comp
-L eSim_NPN Q1
-U 1 1 5CE41586
-P 1850 2350
-F 0 "Q1" H 1750 2400 50  0000 R CNN
-F 1 "eSim_NPN" H 1800 2500 50  0000 R CNN
-F 2 "" H 2050 2450 29  0000 C CNN
-F 3 "" H 1850 2350 60  0000 C CNN
-	1    1850 2350
-	1    0    0    -1
-$EndComp
-$Comp
 L R R5
 U 1 1 5CE418C5
@@
 Connection ~ 1250 2350
 $Comp
-L eSim_NPN Q2
+L eSim_NPN-RESCUE-lm7805 Q2
 U 1 1 5CE41D6C
 P 2650 3350
@@
 $EndComp
 $Comp
-L eSim_NPN Q4
+L eSim_NPN-RESCUE-lm7805 Q4
 U 1 1 5CE41E26
 P 3100 4100
@@
 $EndComp
 $Comp
-L eSim_NPN Q3
+L eSim_NPN-RESCUE-lm7805 Q3
 U 1 1 5CE41EFE
 P 2850 4650
@@
 Connection ~ 2750 5200
 $Comp
-L eSim_NPN Q6
+L eSim_NPN-RESCUE-lm7805 Q6
 U 1 1 5CE424FB
 P 3650 4650
@@
 Connection ~ 3200 5200
 $Comp
-L eSim_NPN Q7
+L eSim_NPN-RESCUE-lm7805 Q7
 U 1 1 5CE427DA
 P 3700 2750
@@
 $EndComp
 $Comp
-L eSim_NPN Q8
+L eSim_NPN-RESCUE-lm7805 Q8
 U 1 1 5CE428D0
 P 3700 3400
@@
 $EndComp
 $Comp
-L eSim_NPN Q12
+L eSim_NPN-RESCUE-lm7805 Q12
 U 1 1 5CE4293A
 P 4350 3000
@@
 $EndComp
 $Comp
-L eSim_NPN Q10
+L eSim_NPN-RESCUE-lm7805 Q10
 U 1 1 5CE43705
 P 4100 2200
@@
 Connection ~ 2200 5200
 $Comp
-L eSim_NPN Q11
+L eSim_NPN-RESCUE-lm7805 Q11
 U 1 1 5CE4439E
 P 4300 4400
@@
 $EndComp
 $Comp
-L eSim_NPN Q13
+L eSim_NPN-RESCUE-lm7805 Q13
 U 1 1 5CE44419
 P 4600 4800
@@
 Connection ~ 4750 3450
 $Comp
-L eSim_NPN Q15
+L eSim_NPN-RESCUE-lm7805 Q15
 U 1 1 5CE463AD
 P 5400 2150
@@
 	5850 2150 5600 2150
 $Comp
-L eSim_NPN Q16
+L eSim_NPN-RESCUE-lm7805 Q16
 U 1 1 5CE4907A
 P 6550 1600
@@
 $EndComp
 $Comp
-L eSim_NPN Q17
+L eSim_NPN-RESCUE-lm7805 Q17
 U 1 1 5CE4942E
 P 7300 1950
@@
 Connection ~ 7300 2650
 Connection ~ 2500 5200
+$Comp
+L eSim_NPN-RESCUE-lm7805 Q1
+U 1 1 5D63A1DF
+P 1850 2350
+F 0 "Q1" H 1750 2400 50  0000 R CNN
+F 1 "eSim_NPN" H 1800 2500 50  0000 R CNN
+F 2 "" H 2050 2450 29  0000 C CNN
+F 3 "" H 1850 2350 60  0000 C CNN
+	1    1850 2350
+	1    0    0    -1
+$EndComp
 $EndSCHEMATC
